File: Duet3_Mainboard_v1.01/CAD/Stepper_Drv.sch (KiCad schematic (older format))
At the start: 276 parts, among them Q1 Q_DUAL_NMOS, Q10 Q_DUAL_NMOS, Q11 Q_DUAL_NMOS, Q12 Q_DUAL_NMOS, Q13 Q_DUAL_NMOS, Q14 Q_DUAL_NMOS, Q15 Q_DUAL_NMOS, Q16 Q_DUAL_NMOS, Q17 Q_DUAL_NMOS, Q18 Q_DUAL_NMOS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

Commit message: BAT40V symbol link changed
Parts:
- D38, D39, D40, D41, D42, D43, D44, D45, D46, D47, D48, D49, D50, D51, D52, D53, D54, D55, D56, D57, D58, D59, D60, D61: symbol Diode:BAT40V -> Duet3:BAT40V
Changed lines of the file:
@@
 EESchema Schematic File Version 4
-LIBS:Duet3_MB-cache
 EELAYER 30 0
 EELAYER END
@@
 	20275 7275 20275 7400
 $Comp
-L Diode:BAT40V D39
+L Duet3:BAT40V D39
 U 1 1 5E98FD6D
 P 5250 2475
@@
 $EndComp
 $Comp
-L Diode:BAT40V D39
+L Duet3:BAT40V D39
 U 2 1 5E993A35
 P 5225 1925
@@
 	19725 1800 20200 1800
 $Comp
-L Diode:BAT40V D38
+L Duet3:BAT40V D38
 U 1 1 643EC1A3
 P 5225 1575
@@
 $EndComp
 $Comp
-L Diode:BAT40V D38
+L Duet3:BAT40V D38
 U 2 1 643EC1AD
 P 5250 2825
@@
 $EndComp
 $Comp
-L Diode:BAT40V D41
+L Duet3:BAT40V D41
 U 1 1 64F6E79A
 P 5275 3825
@@
 $EndComp
 $Comp
-L Diode:BAT40V D40
+L Duet3:BAT40V D40
 U 2 1 64F6E7A4
 P 5275 4150
@@
 $EndComp
 $Comp
-L Diode:BAT40V D40
+L Duet3:BAT40V D40
 U 1 1 64F6E7AE
 P 5250 3050
@@
 $EndComp
 $Comp
-L Diode:BAT40V D41
+L Duet3:BAT40V D41
 U 2 1 64F6E7B8
 P 5250 3350
@@
 	4300 1950 4375 1950
 $Comp
-L Diode:BAT40V D43
+L Duet3:BAT40V D43
 U 1 1 6C4FEF62
 P 12475 2475
@@
 $EndComp
 $Comp
-L Diode:BAT40V D42
+L Duet3:BAT40V D42
 U 2 1 6C4FEF6C
 P 12475 2800
@@
 $EndComp
 $Comp
-L Diode:BAT40V D42
+L Duet3:BAT40V D42
 U 1 1 6C4FEF7F
 P 12450 1575
@@
 $EndComp
 $Comp
-L Diode:BAT40V D43
+L Duet3:BAT40V D43
 U 2 1 6C4FEF89
 P 12525 1925
@@
 $EndComp
 $Comp
-L Diode:BAT40V D45
+L Duet3:BAT40V D45
 U 1 1 6C4FEF93
 P 12500 3825
@@
 $EndComp
 $Comp
-L Diode:BAT40V D45
+L Duet3:BAT40V D45
 U 2 1 6C4FEF9D
 P 12475 3325
@@
 $EndComp
 $Comp
-L Diode:BAT40V D44
+L Duet3:BAT40V D44
 U 1 1 6C4FEFA7
 P 12475 3050
@@
 $EndComp
 $Comp
-L Diode:BAT40V D44
+L Duet3:BAT40V D44
 U 2 1 6C4FEFB1
 P 12525 4150
@@
 $EndComp
 $Comp
-L Diode:BAT40V D51
+L Duet3:BAT40V D51
 U 1 1 6CD10CD8
 P 5100 7400
@@
 $EndComp
 $Comp
-L Diode:BAT40V D50
+L Duet3:BAT40V D50
 U 2 1 6CD10CE2
 P 5100 7725
@@
 $EndComp
 $Comp
-L Diode:BAT40V D50
+L Duet3:BAT40V D50
 U 1 1 6CD10CEC
 P 5075 6500
@@
 $EndComp
 $Comp
-L Diode:BAT40V D51
+L Duet3:BAT40V D51
 U 2 1 6CD10CF6
 P 5075 6850
@@
 $EndComp
 $Comp
-L Diode:BAT40V D53
+L Duet3:BAT40V D53
 U 1 1 6CD10D00
 P 5125 8750
@@
 $EndComp
 $Comp
-L Diode:BAT40V D53
+L Duet3:BAT40V D53
 U 2 1 6CD10D0A
 P 5075 8250
@@
 $EndComp
 $Comp
-L Diode:BAT40V D52
+L Duet3:BAT40V D52
 U 1 1 6CD10D14
 P 5100 7975
@@
 $EndComp
 $Comp
-L Diode:BAT40V D52
+L Duet3:BAT40V D52
 U 2 1 6CD10D1E
 P 5125 9075
@@
 $EndComp
 $Comp
-L Diode:BAT40V D55
+L Duet3:BAT40V D55
 U 1 1 6CFAF296
 P 12525 7400
@@
 $EndComp
 $Comp
-L Diode:BAT40V D54
+L Duet3:BAT40V D54
 U 2 1 6CFAF2A0
 P 12525 7725
@@
 $EndComp
 $Comp
-L Diode:BAT40V D54
+L Duet3:BAT40V D54
 U 1 1 6CFAF2AA
 P 12500 6500
@@
 $EndComp
 $Comp
-L Diode:BAT40V D55
+L Duet3:BAT40V D55
 U 2 1 6CFAF2B4
 P 12500 6850
@@
 $EndComp
 $Comp
-L Diode:BAT40V D57
+L Duet3:BAT40V D57
 U 1 1 6CFAF2BE
 P 12550 8750
@@
 $EndComp
 $Comp
-L Diode:BAT40V D57
+L Duet3:BAT40V D57
 U 2 1 6CFAF2C8
 P 12525 8250
@@
 $EndComp
 $Comp
-L Diode:BAT40V D56
+L Duet3:BAT40V D56
 U 1 1 6CFAF2D2
 P 12525 7975
@@
 $EndComp
 $Comp
-L Diode:BAT40V D56
+L Duet3:BAT40V D56
 U 2 1 6CFAF2DC
 P 12550 9075
@@
 $EndComp
 $Comp
-L Diode:BAT40V D59
+L Duet3:BAT40V D59
 U 1 1 6CFAF2E6
 P 19925 7400
@@
 $EndComp
 $Comp
-L Diode:BAT40V D58
+L Duet3:BAT40V D58
 U 2 1 6CFAF2F0
 P 19925 7725
@@
 $EndComp
 $Comp
-L Diode:BAT40V D58
+L Duet3:BAT40V D58
 U 1 1 6CFAF2FA
 P 19900 6500
@@
 $EndComp
 $Comp
-L Diode:BAT40V D59
+L Duet3:BAT40V D59
 U 2 1 6CFAF304
 P 19900 6850
@@
 $EndComp
 $Comp
-L Diode:BAT40V D61
+L Duet3:BAT40V D61
 U 1 1 6CFAF30E
 P 19950 8750
@@
 $EndComp
 $Comp
-L Diode:BAT40V D61
+L Duet3:BAT40V D61
 U 2 1 6CFAF318
 P 19925 8250
@@
 $EndComp
 $Comp
-L Diode:BAT40V D60
+L Duet3:BAT40V D60
 U 1 1 6CFAF322
 P 19925 7975
@@
 $EndComp
 $Comp
-L Diode:BAT40V D60
+L Duet3:BAT40V D60
 U 2 1 6CFAF32C
 P 19950 9075
@@
 $EndComp
 $Comp
-L Diode:BAT40V D48
+L Duet3:BAT40V D48
 U 2 1 6CA6C814
 P 19950 4150
@@
 $EndComp
 $Comp
-L Diode:BAT40V D48
+L Duet3:BAT40V D48
 U 1 1 6CA6C80A
 P 19925 3050
@@
 $EndComp
 $Comp
-L Diode:BAT40V D49
+L Duet3:BAT40V D49
 U 2 1 6CA6C800
 P 19900 3325
@@
 $EndComp
 $Comp
-L Diode:BAT40V D49
+L Duet3:BAT40V D49
 U 1 1 6CA6C7F6
 P 19950 3825
@@
 $EndComp
 $Comp
-L Diode:BAT40V D47
+L Duet3:BAT40V D47
 U 2 1 6CA6C7EC
 P 19900 1925
@@
 $EndComp
 $Comp
-L Diode:BAT40V D46
+L Duet3:BAT40V D46
 U 1 1 6CA6C7E2
 P 19900 1575
@@
 $EndComp
 $Comp
-L Diode:BAT40V D46
+L Duet3:BAT40V D46
 U 2 1 6CA6C7D8
 P 19925 2800
@@
 $EndComp
 $Comp
-L Diode:BAT40V D47
+L Duet3:BAT40V D47
 U 1 1 6CA6C7CE
 P 19925 2475
